Commit message: Use real Franka meshes in combined URDF + add third-person render tool
- generate_combined_urdf.py: replace primitive cylinder/box arm geometry with the
  official franka_description visual (.dae) + collision (.stl) meshes for link0-7,
  so the bimanual eval renders real Franka arms instead of blobs. Hand mount is
  now configurable via MOUNT_RPY/MOUNT_XYZ env vars (90-deg bracket TBD).
- Vendor franka_description/meshes (from the Isaac URDF-importer assets).
- Regenerate franka_orca_{left,right}.urdf with the real meshes.
- eval_utils/render_thirdperson.py: headless third-person render harness for
  visually validating the scene/arm layout against the real rig.
- .gitignore: ignore local output/ and *.bak backups.

Co-Authored-By: Claude Opus 4.8 (1M context) <noreply@anthropic.com>

File: sim_envs/assets/franka_orca_left.urdf (robot description, URDF)
Before this commit: robot franka_orca_left, 51 links, 50 joints
Links:
- link panda_link0: geometry collision mesh filename=franka_description/meshes/collision/link0.stl; visual mesh filename=franka_description/meshes/visual/link0.dae
- link panda_link1: geometry collision mesh filename=franka_description/meshes/collision/link1.stl; visual mesh filename=franka_description/meshes/visual/link1.dae
- link panda_link2: geometry collision mesh filename=franka_description/meshes/collision/link2.stl; visual mesh filename=franka_description/meshes/visual/link2.dae
- link panda_link3: geometry collision mesh filename=franka_description/meshes/collision/link3.stl; visual mesh filename=franka_description/meshes/visual/link3.dae
- link panda_link4: geometry collision mesh filename=franka_description/meshes/collision/link4.stl; visual mesh filename=franka_description/meshes/visual/link4.dae
- link panda_link5: geometry collision mesh filename=franka_description/meshes/collision/link5.stl; visual mesh filename=franka_description/meshes/visual/link5.dae
- link panda_link6: geometry collision mesh filename=franka_description/meshes/collision/link6.stl; visual mesh filename=franka_description/meshes/visual/link6.dae
- link panda_link7: geometry collision mesh filename=franka_description/meshes/collision/link7.stl; visual mesh filename=franka_description/meshes/visual/link7.dae

File: sim_envs/assets/franka_orca_right.urdf (robot description, URDF)
Before this commit: robot franka_orca_right, 51 links, 50 joints
Links:
- link panda_link0: geometry collision mesh filename=franka_description/meshes/collision/link0.stl; visual mesh filename=franka_description/meshes/visual/link0.dae
- link panda_link1: geometry collision mesh filename=franka_description/meshes/collision/link1.stl; visual mesh filename=franka_description/meshes/visual/link1.dae
- link panda_link2: geometry collision mesh filename=franka_description/meshes/collision/link2.stl; visual mesh filename=franka_description/meshes/visual/link2.dae
- link panda_link3: geometry collision mesh filename=franka_description/meshes/collision/link3.stl; visual mesh filename=franka_description/meshes/visual/link3.dae
- link panda_link4: geometry collision mesh filename=franka_description/meshes/collision/link4.stl; visual mesh filename=franka_description/meshes/visual/link4.dae
- link panda_link5: geometry collision mesh filename=franka_description/meshes/collision/link5.stl; visual mesh filename=franka_description/meshes/visual/link5.dae
- link panda_link6: geometry collision mesh filename=franka_description/meshes/collision/link6.stl; visual mesh filename=franka_description/meshes/visual/link6.dae
- link panda_link7: geometry collision mesh filename=franka_description/meshes/collision/link7.stl; visual mesh filename=franka_description/meshes/visual/link7.dae
