Commit message: Enhance Franka + Orca bimanual simulation fidelity and validation
- Implemented `sanitize_inertials()` to assign valid mass and inertia to massless fingertip/root links in URDF, preventing instability in dynamics.
- Updated `FrankaOrcaBimanualEnv` to ensure actions are treated as absolute targets, correcting the action application logic.
- Refined action term order in `ActionsCfg` to match training layout, ensuring consistency in joint control.
- Added manipulable objects (grocery bag, container, tube, round item) to the scene, aligning with training data.
- Adjusted hand actuator parameters (stiffness, damping, effort limit) for improved grasp tracking.
- Created validation tooling (`inspect_joints.py`) to verify joint setup against training contract, including action path and joint order checks.
- Documented changes and validation process in `SIM_VALIDATION_AND_SCENE.md`.
- Added SLURM scripts for joint inspection and full closed-loop evaluation.

File: sim_envs/assets/franka_orca_left.urdf (robot description, URDF)
Before this commit: robot franka_orca_left, 51 links, 50 joints
Links:
- link left_index_fingertip: mass 0.0 -> 0.01
- link left_middle_fingertip: mass 0.0 -> 0.01
- link left_pinky_fingertip: mass 0.0 -> 0.01
- link left_ring_fingertip: mass 0.0 -> 0.01
- link left_root: mass 0.0 -> 0.01
- link left_thumb_fingertip: mass 0.0 -> 0.01

File: sim_envs/assets/franka_orca_right.urdf (robot description, URDF)
Before this commit: robot franka_orca_right, 51 links, 50 joints
Links:
- link right_index_fingertip: mass 0.0 -> 0.01
- link right_middle_fingertip: mass 0.0 -> 0.01
- link right_pinky_fingertip: mass 0.0 -> 0.01
- link right_ring_fingertip: mass 0.0 -> 0.01
- link right_root: mass 0.0 -> 0.01
- link right_thumb_fingertip: mass 0.0 -> 0.01

Commit message: Sim fidelity, camera tuning, and eval/debug tooling
Simulation (franka_orca_bimanual):
- Add high-friction grip material to table and graspable objects;
  rely on friction_combine_mode="max" so grasps hold.
- Separate camera viewpoints: oak-d front top-down pose vs aria
  wide-FOV ego pose (aria focal 20->8); both at native train
  resolutions (aria 640x480, oakd 960x540) @ 50 Hz.
- Add visual-only floor + back-wall backdrop.
- Fix left-arm joint convention: ARM_SIM_FROM_REAL remap (+/-pi on
  j4/j6) with real_arm_to_sim / sim_arm_to_real helpers, applied to
  both actions and proprioception in the bimanual eval loop.
- Fix mirrored left-wrist joint axis in franka_orca_left.urdf and the
  generate_combined_urdf mirroring logic.

Tooling:
- New eval/debug scripts: grasp_test, render_cameras, replay_h5,
  show_hands, with matching euler sbatch wrappers.
- Action-chunk logging in the AR inference server (franka_orca_bimanual).

Docs: expand SIM_VALIDATION_AND_SCENE with grasp/camera/joint-convention
notes and a pre-retrain checklist.

File: sim_envs/assets/franka_orca_left.urdf (robot description, URDF)
Before this commit: robot franka_orca_left, 51 links, 50 joints
Joints:
- joint left_wrist: axis -1.0 0.0 0.0 -> 1.0 0.0 0.0

Commit message: Fix EE orientation convention: quaternion is scalar-first (A @ wxyz), not xyzw
The prior commit read the arm-pose quaternion scalar-LAST (xyzw); that is a ~142deg
wrist error that twists both hands inward and makes them interpenetrate at convergence
frames (e.g. t=1960) while staying IK-reachable (so it hid in the residual). The correct
flange orientation is R_flange = A @ R_wxyz, reading the quaternion scalar-first and
pre-multiplying A = 135deg about (-1,1,1)/sqrt3. This is the only convention that keeps the
two hands non-colliding (min hand-hand 229mm vs 8.6mm) AND pointing down at the table (100%
of grasp frames vs 39%); verified by render at t=1960 (collision gone, hands point down).

- export_xyzw_full.py: A @ wxyz convention + continuity-preserving re-seed fallback.
- generate_combined_urdf.py: revert left Gavin-mount rpy to the original 1.832292 0 3.141593
  (best mirror of the right hand under the correct orientation); the mid-session 'option Y'
  was compensating the orientation bug and is wrong. Regenerate franka_orca_left.urdf.
- docs/EE_POSE_AND_IK_PIPELINE.md: corrected convention + known right-arm IK-tracking segment.

Known remaining: right-arm warm-start IK gets trapped on frames ~1670-1905 (reachable from
fresh seeds); needs branch-tracking IK or a per-arm A refinement.

File: sim_envs/assets/franka_orca_left.urdf (robot description, URDF)
Before this commit: robot franka_orca_left, 52 links, 51 joints
Joints:
- joint gavin_mount_to_left_hand: origin xyz=0.006220897 -0.03045047 0.08067889 rpy=1.403854 -0.047154 3.052323 -> xyz=0.006220897 -0.03045047 0.08067889 rpy=1.832292 0.0 3.141593

Commit message: Revert "Fix EE orientation convention: quaternion is scalar-first (A @ wxyz), not xyzw"
This reverts commit bc62209a02d20a874530d6025ecc003b9d57a049.

File: sim_envs/assets/franka_orca_left.urdf (robot description, URDF)
Before this commit: robot franka_orca_left, 52 links, 51 joints
Joints:
- joint gavin_mount_to_left_hand: origin xyz=0.006220897 -0.03045047 0.08067889 rpy=1.832292 0.0 3.141593 -> xyz=0.006220897 -0.03045047 0.08067889 rpy=1.403854 -0.047154 3.052323

Commit message: Trim left hand mount 4cm along mount-local Y (user-confirmed against renders)

File: sim_envs/assets/franka_orca_left.urdf (robot description, URDF)
Before this commit: robot franka_orca_left, 52 links, 51 joints
Joints:
- joint gavin_mount_to_left_hand: origin xyz=0.006220897 -0.03045047 0.08067889 rpy=1.403854 -0.047154 3.052323 -> xyz=0.006220897 -0.07045047 0.08067889 rpy=1.403854 -0.047154 3.052323
