Commit message: Decode franka_orca arm fields as EE poses; fix left hand URDF; add IK solver
qpos_arm_*/actions_arm_* 7-vectors are end-effector poses
[x,y,z,qx,qy,qz,qw] (flange position in base frame; quaternion scalar-last/XYZW),
not joint angles; they must be IK'd to Panda joint targets to drive the robot.

- Add EE-pose -> joint IK solver: eval_utils/export_xyzw_full.py.
- Fix left hand: build from the proper chirality hand (sim_envs/assets/
  orcahand_left.urdf) instead of the invalid in-script mirror, and correct the left
  Gavin mount (y-mirror of right then +180deg about root-local Y) so it closes the
  right way; regenerate franka_orca_{left,right}.urdf.
- Document the decode + IK pipeline in docs/EE_POSE_AND_IK_PIPELINE.md.
- Ignore generated artifacts (npz, h5, mp4, archive/).

File: sim_envs/assets/franka_orca_right.urdf (robot description, URDF)
Before this commit: robot franka_orca_right, 51 links, 50 joints
Links:
- added link right_gavin_mount, mass 0.05; visual box size=0.030 0.030 0.090; visual box size=0.065 0.055 0.012
Joints:
- removed joint panda_link8_to_right_hand
- added joint gavin_mount_to_right_hand: type fixed, parent right_gavin_mount, child right_root, origin xyz=0.006220897 0.03045047 0.08067889 rpy=1.737739 0.047154 -0.089270
- added joint panda_link8_to_right_gavin_mount: type fixed, parent panda_link8, child right_gavin_mount, origin xyz=0 0 0 rpy=0 0 1.5707963
- joint panda_joint6: limit lower=-0.0175 upper=3.7525 effort=87.0 velocity=2.175 -> lower=-1.0 upper=3.7525 effort=87.0 velocity=2.175

File: sim_envs/assets/orcahand_left.urdf (robot description, URDF)
Before this commit: robot franka_orca_left, 52 links, 51 joints
Links:
- removed link left_gavin_mount
- removed link panda_link0
- removed link panda_link1
- removed link panda_link2
- removed link panda_link3
- removed link panda_link4
- removed link panda_link5
- removed link panda_link6
- removed link panda_link7
- removed link panda_link8
- link left_index_fingertip: mass 0.01 -> 0.0
- link left_index_ip: geometry collision mesh filename=package://orcahand_description/assets/urdf/collision/index_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 scale=-1 1 1; collision mesh filename=package://orcahand_description/assets/urdf/collision/index_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 scale=-1 1 1
- link left_index_mp: geometry collision mesh filename=package://orcahand_description/assets/urdf/collision/index_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 scale=-1 1 1; visual mesh filename=package://orcahand_description/assets/urdf/visual/index_mp_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 scale=-1 1 1
- link left_index_pp: geometry collision mesh filename=package://orcahand_description/assets/urdf/collision/index_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 scale=-1 1 1; collision mesh filename=package://orcahand_description/assets/urdf/collision/index_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 scale=-1 1 1
- link left_middle_fingertip: mass 0.01 -> 0.0
- link left_middle_ip: geometry collision mesh filename=package://orcahand_description/assets/urdf/collision/middle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 scale=-1 1 1; collision mesh filename=package://orcahand_description/assets/urdf/collision/middle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 scale=-1 1 1
- link left_middle_mp: geometry collision mesh filename=package://orcahand_description/assets/urdf/collision/middle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 scale=-1 1 1; visual mesh filename=package://orcahand_description/assets/urdf/visual/middle_mp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 scale=-1 1 1
- link left_middle_pp: geometry collision mesh filename=package://orcahand_description/assets/urdf/collision/middle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 scale=-1 1 1; collision mesh filename=package://orcahand_description/assets/urdf/collision/middle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 scale=-1 1 1
- link left_palm: geometry collision mesh filename=package://orcahand_description/assets/urdf/collision/palm_m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 scale=-1 1 1; collision mesh filename=package://orcahand_description/assets/urdf/collision/palm_s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 scale=-1 1 1
- link left_pinky_fingertip: mass 0.01 -> 0.0
- link left_pinky_ip: geometry collision mesh filename=package://orcahand_description/assets/urdf/collision/pinky_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 scale=-1 1 1; collision mesh filename=package://orcahand_description/assets/urdf/collision/pinky_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 scale=-1 1 1
- link left_pinky_mp: geometry collision mesh filename=package://orcahand_description/assets/urdf/collision/pinky_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 scale=-1 1 1; visual mesh filename=package://orcahand_description/assets/urdf/visual/pinky_mp_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 scale=-1 1 1
- link left_pinky_pp: geometry collision mesh filename=package://orcahand_description/assets/urdf/collision/pinky_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 scale=-1 1 1; collision mesh filename=package://orcahand_description/assets/urdf/collision/pinky_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 scale=-1 1 1
- link left_ring_fingertip: mass 0.01 -> 0.0
- link left_ring_ip: geometry collision mesh filename=package://orcahand_description/assets/urdf/collision/ring_i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 scale=-1 1 1; collision mesh filename=package://orcahand_description/assets/urdf/collision/ring_i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 scale=-1 1 1
- link left_ring_mp: geometry collision mesh filename=package://orcahand_description/assets/urdf/collision/ring_m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 scale=-1 1 1; visual mesh filename=package://orcahand_description/assets/urdf/visual/ring_mp_m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 scale=-1 1 1
- link left_ring_pp: geometry collision mesh filename=package://orcahand_description/assets/urdf/collision/ring_p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 scale=-1 1 1; collision mesh filename=package://orcahand_description/assets/urdf/collision/ring_p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 scale=-1 1 1
- link left_root: mass 0.01 -> 0.0
- link left_thumb_dp: geometry collision mesh filename=package://orcahand_description/assets/urdf/collision/thumb_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 scale=-1 1 1; collision mesh filename=package://orcahand_description/assets/urdf/collision/thumb_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 scale=-1 1 1
- link left_thumb_fingertip: mass 0.01 -> 0.0
- link left_thumb_ip: geometry collision mesh filename=package://orcahand_description/assets/urdf/collision/thumb_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 scale=-1 1 1; collision mesh filename=package://orcahand_description/assets/urdf/collision/thumb_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 scale=-1 1 1
- link left_thumb_mp: geometry collision mesh filename=package://orcahand_description/assets/urdf/collision/thumb_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 scale=-1 1 1; visual mesh filename=package://orcahand_description/assets/urdf/visual/thumb_mp_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 scale=-1 1 1
- link left_thumb_pp: geometry collision mesh filename=package://orcahand_description/assets/urdf/collision/thumb_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 scale=-1 1 1; visual mesh filename=package://orcahand_description/assets/urdf/visual/thumb_pp_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 scale=-1 1 1
- link left_tower: geometry collision mesh filename=package://orcahand_description/assets/urdf/collision/tower_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 scale=-1 1 1; collision mesh filename=package://orcahand_description/assets/urdf/collision/tower_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 scale=-1 1 1
Joints:
- removed joint gavin_mount_to_left_hand
- removed joint panda_joint1
- removed joint panda_joint2
- removed joint panda_joint3
- removed joint panda_joint4
- removed joint panda_joint5
- removed joint panda_joint6
- removed joint panda_joint7
- removed joint panda_joint8
- removed joint panda_link8_to_left_gavin_mount
